File: pcf8563-breakout.kicad_sch (KiCad schematic)
At the start: 32 parts, among them J1 Conn_01x04_Socket, J2 Conn_01x03_Pin, J3 Conn_01x04_Socket, J4 Conn_01x07_Socket, U1 PCF8563T, U2 SHT4x, U3 LSM6DSVTR, U4 IIS2MDCTR, X1 Q13FC1350000400

Commit message: feat: updates and journal
Parts:
- removed C6: 220nF, PCM_JLCPCB:C_0603, symbol PCM_JLCPCB-Capacitors:0603,220nF
- removed C7, C8: 100nF, PCM_JLCPCB:C_0402, symbol PCM_JLCPCB-Capacitors:0402,100nF,(2)
- removed C9: 10uF, PCM_JLCPCB:C_0603, symbol PCM_JLCPCB-Capacitors:0603,10uF,(2)
- removed R1, R2: 2.2kΩ, PCM_JLCPCB:R_0603, symbol PCM_JLCPCB-Resistors:0603,2.2kΩ
- removed R4, R5: 2.2kΩ, PCM_JLCPCB:R_0402, symbol PCM_JLCPCB-Resistors:0402,2.2kΩ
- removed U4: IIS2MDCTR, easyeda2kicad:LGA-12_L2.0-W2.0-P0.50-TL, symbol easyeda2kicad:IIS2MDCTR
- added C6: 2.2uF, PCM_JLCPCB:C_0603, symbol PCM_JLCPCB-Capacitors:0603,2.2uF
- added C7, C8: 1uF, PCM_JLCPCB:C_0603, symbol PCM_JLCPCB-Capacitors:0603,1uF
- added Q1, Q2: BSS138W, PCM_JLCPCB:Q_SOT-323, symbol PCM_JLCPCB-Transistors:NMOS,BSS138W
- added R1, R2: 10kΩ, PCM_JLCPCB:R_0402, symbol PCM_JLCPCB-Resistors:0402,10kΩ
- added R6: 10kΩ, PCM_JLCPCB:R_0402x4, symbol PCM_JLCPCB-Resistors:0402x4,10kΩ
- added U4: QMC6309, easyeda2kicad:X1-WLB0808-4_L0.8-W0.8-P0.40-TL, symbol easyeda2kicad:QMC6309
- added U5: XC6206P332MR, PCM_JLCPCB:SOT-23-3_L2.9-W1.6-P1.90-LS2.8-BR, symbol PCM_JLCPCB-Power:LDO, 3.3V, 0.2A
- U3: value LSM6DSVTR -> LSM6DSVQTR
Connections:
- net GND: now also C6.2, C7.2, C8.2, U4.A1 (VSS), U5.1 (GND)
- net MSCL: now also Q2.2 (S), R6.6
- net MSDA: now also Q1.2 (S), R6.7
- net VDD: now also Q1.1 (G), Q2.1 (G), R1.2, R2.1, R6.2, R6.3
- net at JP1.2 (B): now also R1.1
- net at JP2.2 (B): now also R2.2
- new net: C7.1, U5.3 (VIN)
- new net +3.3V: C6.1, C8.1, R6.1, R6.4, U4.B1 (VDD), U5.2 (VOUT)
- new net QMSCL: Q2.3 (D), R6.5, U4.A2 (SCL)
- new net QMSDA: Q1.3 (D), R6.8, U4.B2 (SDA)

Commit message: fix: readme
Parts:
- removed C1, C3, C4, C5: 100nF, PCM_JLCPCB:C_0603, symbol PCM_JLCPCB-Capacitors:0603,100nF
- removed C2: 22pF, PCM_JLCPCB:C_0603, symbol PCM_JLCPCB-Capacitors:0603,22pF
- removed C7, C8: 1uF, PCM_JLCPCB:C_0603, symbol PCM_JLCPCB-Capacitors:0603,1uF
- removed R6: 10kΩ, PCM_JLCPCB:R_0402x4, symbol PCM_JLCPCB-Resistors:0402x4,10kΩ
- added C1, C3, C4, C5: 100nF, PCM_JLCPCB:C_0402, symbol PCM_JLCPCB-Capacitors:0402,100nF,(2)
- added C2: 22pF, PCM_JLCPCB:C_0402, symbol PCM_JLCPCB-Capacitors:0402,22pF
- added C7, C8: 1uF, PCM_JLCPCB:C_0402, symbol PCM_JLCPCB-Capacitors:0402,1uF
- added J5: Conn_01x01_Pin, Connector_PinHeader_1.27mm:PinHeader_1x01_P1.27mm_Vertical, symbol Connector:Conn_01x01_Pin
- added R4: 10kΩ, PCM_JLCPCB:R_0402x4, symbol PCM_JLCPCB-Resistors:0402x4,10kΩ
Connections:
- net +3.3V: now also C7.1, R4.3, R4.4
- net GND: now also C1.2, C2.2, C3.2, C4.1, C5.1, C7.2, C8.2
- net MSCL: now also R4.7
- net MSDA: now also R4.8
- net QMSCL: now also R4.5
- net QMSDA: now also R4.6
- net VDD: now also C3.1, C4.2, C5.2, R4.1, R4.2
- net VIN: now also C1.1
- net at U1.1 (OSCI), X1.1: now also C2.1
- net at U5.3 (VIN): now also C8.1, J5.1 (Pin_1)
Other:
- note added: "IMU"
- note added: "IMU + Mag Connectors"
- note added: "Magnetometer + Level Shifting"
- note removed: "IMU + Mag Connectors & Pullups"
- note removed: "IMU and Magnetometer"
- moved on the sheet: BT1, C6, D1, D2, D3, J1, J2, J3, J4, JP1, JP2, JP3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
