File: pcf8563-breakout.kicad_pcb (KiCad board)
At the start: 4 copper layers, 29.5 x 16.8 mm, 32 parts, among them J1 Conn_01x04_Socket, J2 Conn_01x03_Pin, J3 Conn_01x04_Socket, J4 Conn_01x07_Socket, U1 PCF8563T, U2 SHT4x, U3 LSM6DSVTR, U4 IIS2MDCTR, X1 Q13FC1350000400

Commit message: feat: updates and journal
Parts:
- removed C9: 10uF, PCM_JLCPCB:C_0603
- removed R5: 2.2kΩ, PCM_JLCPCB:R_0402
- added J5: Conn_01x01_Pin, Connector_PinHeader_1.27mm:PinHeader_1x01_P1.27mm_Vertical, F.Cu at (127.2, 103.6)
- added Q1: BSS138W, PCM_JLCPCB:Q_SOT-323, F.Cu at (127.5, 106.0)
- added Q2: BSS138W, PCM_JLCPCB:Q_SOT-323, F.Cu at (130.6, 111.7)
- added U5: XC6206P332MR, PCM_JLCPCB:SOT-23-3_L2.9-W1.6-P1.90-LS2.8-BR, F.Cu at (127.5, 109.2)
- C1, C2, C3, C4, C5: footprint PCM_JLCPCB:C_0603 -> PCM_JLCPCB:C_0402
- C6: value 220nF -> 2.2uF
- C7, C8: value 100nF -> 1uF
- R1, R2: value 2.2kΩ -> 10kΩ; footprint PCM_JLCPCB:R_0603 -> PCM_JLCPCB:R_0402
- R4: value 2.2kΩ -> 10kΩ; footprint PCM_JLCPCB:R_0402 -> PCM_JLCPCB:R_0402x4
- U3: value LSM6DSVTR -> LSM6DSVQTR
- U4: value IIS2MDCTR -> QMC6309; footprint easyeda2kicad:LGA-12_L2.0-W2.0-P0.50-TL -> easyeda2kicad:X1-WLB0808-4_L0.8-W0.8-P0.40-TL
- moved JP5 6.50 mm to (133.6, 102.6)
- moved C6 5.99 mm to (134.0, 111.6), turned to -90 degrees
- moved U4 3.31 mm to (132.8, 111.5)
- moved C7 2.73 mm to (129.9, 109.3), turned to -90 degrees
- moved JP2 1.78 mm to (150.3, 107.4)
- moved C8 1.77 mm to (126.0, 107.7)
- moved D1 1.75 mm to (143.8, 108.6)
- moved C2 1.14 mm to (140.6, 109.6)
- moved JP4 1.12 mm to (131.3, 102.6)
- moved C1 1.10 mm to (146.1, 109.3), turned to 90 degrees
- moved X1 1.02 mm to (139.0, 111.1)
- moved D2 0.88 mm to (148.6, 109.6), turned to 0 degrees
- moved R4 0.88 mm to (130.4, 107.0)
- moved U1 0.85 mm to (143.8, 113.1)
- moved C3 0.81 mm to (129.3, 101.3)
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Connections:
- C6 pad 1: GND -> +3.3V
- C6 pad 2: Net-(U4-C1) -> GND
- C7 pad 1: VDD -> +3.3V
- C8 pad 1: VDD -> Net-(J5-Pin_1)
- R4 pad 2: /MSDA -> VDD
Routing:
- net +3.3V: track 0.00 -> 15.4 mm, vias 0 -> 2
- net /QMSDA: track 0.00 -> 13.9 mm, vias 0 -> 2
- net /QMSCL: track 0.00 -> 7.58 mm
- net Net-(J5-Pin_1): track 0.00 -> 7.33 mm
- net VDD: track 28.5 -> 21.3 mm, vias 12 -> 10
- net GND: track 29.7 -> 25.7 mm, vias 17 -> 12
- net /SCL: track 49.7 -> 45.6 mm, vias 3 -> 4
- net /SDA: track 47.9 -> 44.0 mm
- net /VIN: track 8.53 -> 5.36 mm
- net /MSDA: track 6.19 -> 8.44 mm
- net /INT_I: track 10.4 -> 8.88 mm
- net Net-(U4-C1): track 1.46 -> 0.00 mm
- net /MSCL: track 14.6 -> 13.3 mm
- net /INT: track 13.7 -> 14.4 mm
- net Net-(U1-OSCI): track 3.74 -> 3.10 mm
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Other:
- board text added: "VB+"

Commit message: feat: readme
Routing:
- net Net-(BT1-+): track 6.61 -> 2.04 mm
Changed lines of the file:
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@@
 		)
 		(embedded_fonts no)
-		(model "${KICAD9_3DMODEL_DIR}/Connector_PinHeader_1.27mm.3dshapes/PinHeader_1x01_P1.27mm_Vertical.step"
-			(offset
-				(xyz 0 0 0)
-			)
-			(scale
-				(xyz 1 1 1)
-			)
-			(rotate
-				(xyz 0 0 0)
-			)
-		)
 	)
 	(footprint "PCM_JLCPCB:C_0402"
@@
 	)
 	(segment
-		(start 151.7 109.6)
+		(start 150.425 108.825)
 		(end 149.65 109.6)
 		(width 0.3)
@@
 		(net 1)
 	)
-	(segment
-		(start 153.1 108.2)
-		(end 151.7 109.6)
-		(width 0.3)
-		(layer "F.Cu")
-		(net 1)
-	)
 	(via
-		(at 153.1 108.2)
+		(at 150.425 108.825)
 		(size 0.6)
 		(drill 0.3)
@@
 	)
 	(segment
-		(start 150.6 108)
-		(end 152.9 108)
+		(start 150.654702 108.054702)
+		(end 150.6 108)
+		(width 0.3)
+		(layer "B.Cu")
+		(net 1)
+	)
+	(segment
+		(start 150.654702 108.595298)
+		(end 150.654702 108.054702)
 		(width 0.3)
 		(layer "B.Cu")
@@
 	)
 	(segment
-		(start 152.9 108)
-		(end 153.1 108.2)
+		(start 150.425 108.825)
+		(end 150.654702 108.595298)
 		(width 0.3)
 		(layer "B.Cu")

Commit message: feat: pcb fix
Routing:
- net GND: track 25.7 -> 22.1 mm, vias 12 -> 13
Changed lines of the file:
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@@
 			(at 0 -3.98 0)
 			(layer "F.SilkS")
+			(hide yes)
 			(effects
 				(font
@@
 		(at 132.8 111.5 180)
 		(property "Reference" "U4"
-			(at 0 -1.7 0)
+			(at 0.1 -1.2 0)
 			(layer "F.SilkS")
 			(effects
 				(font
-					(size 1 1)
-					(thickness 0.15)
+					(size 0.8 0.8)
+					(thickness 0.1)
 				)
 			)
@@
 		(tags "Through hole pin header THT 1x01 1.27mm single row")
 		(property "Reference" "J5"
-			(at 0 -1.745 0)
+			(at 1.9 0 0)
 			(layer "F.SilkS")
+			(hide yes)
 			(effects
 				(font
@@
 		(at 133.9 106.5)
 		(property "Reference" "U3"
-			(at 0 -2.2 0)
+			(at 0 -2 0)
 			(layer "F.SilkS")
 			(effects
 				(font
-					(size 1 1)
-					(thickness 0.15)
+					(size 0.8 0.8)
+					(thickness 0.1)
 				)
 			)
@@
 	)
 	(segment
-		(start 139.105 115.005)
-		(end 138.8 114.7)
-		(width 0.2)
-		(layer "F.Cu")
-		(net 2)
-	)
-	(segment
-		(start 129.7 109.6)
-		(end 129.29 109.6)
-		(width 0.3)
-		(layer "F.Cu")
-		(net 2)
-	)
-	(segment
 		(start 135.1 108.5)
 		(end 134.3 108.5)
@@
 	)
 	(segment
+		(start 141.325 115.005)
+		(end 139.105 115.005)
+		(width 0.3)
+		(layer "F.Cu")
+		(net 2)
+	)
+	(segment
 		(start 134.3 108.3)
 		(end 134.3 108.5)
@@
 	)
 	(segment
-		(start 129.29 109.6)
-		(end 128.74 110.15)
-		(width 0.3)
-		(layer "F.Cu")
-		(net 2)
-	)
-	(segment
 		(start 137.92 114.7)
 		(end 137.82 114.8)
@@
 	)
 	(segment
+		(start 129.9 109.8)
+		(end 129.09 109.8)
+		(width 0.3)
+		(layer "F.Cu")
+		(net 2)
+	)
+	(segment
 		(start 133.34 111.7)
 		(end 134 112.36)
@@
 	)
 	(segment
-		(start 141.325 115.005)
-		(end 139.105 115.005)
-		(width 0.2)
-		(layer "F.Cu")
-		(net 2)
-	)
-	(segment
-		(start 144.4 106.3)
-		(end 146.1 108)
+		(start 139.105 115.005)
+		(end 138.8 114.7)
 		(width 0.3)
 		(layer "F.Cu")
@@
 	)
 	(segment
-		(start 143.1 104.9)
-		(end 143.9 104.9)
+		(start 129.09 109.8)
+		(end 128.74 110.15)
 		(width 0.3)
 		(layer "F.Cu")
@@
 	)
 	(segment
-		(start 134.9 112.15)
-		(end 134.65 112.4)
+		(start 143.1 104.9)
+		(end 143.9 104.9)
 		(width 0.3)
 		(layer "F.Cu")
@@
 	)
 	(segment
-		(start 143.4 106.3)
-		(end 144.4 106.3)
+		(start 134.9 112.15)
+		(end 134.65 112.4)
 		(width 0.3)
 		(layer "F.Cu")
@@
 	)
 	(segment
-		(start 129.9 109.8)
-		(end 129.7 109.6)
-		(width 0.3)
-		(layer "F.Cu")
-		(net 2)
-	)
-	(segment
 		(start 143.1 106)
 		(end 143.1 104.9)
@@
 	)
 	(via
+		(at 146.1 108)
+		(size 0.6)
+		(drill 0.3)
+		(layers "F.Cu" "B.Cu")
+		(net 2)
+	)
+	(via
 		(at 140.5 108.32)
 		(size 0.6)
@@
 	)
 	(segment
-		(start 143.8 109.65)
-		(end 145.95 109.65)
+		(start 146.1 111.02)
+		(end 146.275 111.195)
 		(width 0.3)
 		(layer "F.Cu")
@@
 	)
 	(segment
-		(start 146.1 111.02)
-		(end 146.275 111.195)
+		(start 143.95 109.8)
+		(end 146.1 109.8)
 		(width 0.3)
 		(layer "F.Cu")
@@
 	)
 	(segment
-		(start 147.35 109.8)
-		(end 147.55 109.6)
+		(start 143.8 109.65)
+		(end 143.95 109.8)
 		(width 0.3)
 		(layer "F.Cu")
@@
 	)
 	(segment
-		(start 145.95 109.65)
-		(end 146.1 109.8)
+		(start 147.35 109.8)
+		(end 147.55 109.6)
 		(width 0.3)
 		(layer "F.Cu")
